File: files/pcb/main.kicad_sch (KiCad schematic)
At the start: 48 parts, among them J1 Power, J10 main row, J11 main col, J12 main row, J13 5V RGB, J14 SignalB, J15 Rotray Encoder, J16 main col, J17 main row, J18 Elite L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

Commit message: renew files and pics
Parts:
- added D1: 1N4148_TS, DreaM117er-keebLibrary:D_DO-35_SOD27_P7.62mm_Horizontal, symbol DreaM117er_Library:DS_1N4148_TS
- added H1, H2: M2, MountingHole:MountingHole_2.2mm_M2, symbol Mechanical:MountingHole
- added H7, H8, H9: edge, Marby_kbd_footprint-main:Breakaway_Tabs, symbol Mechanical:MountingHole
- added J1: LTRRS, DreaM117er-keebLibrary:PinHeader_1x03_P2.54mm_Vertical, symbol Connector:Conn_01x03_Pin
- added J10: row, DreaM117er-keebLibrary:PinHeader_1x01_P2.54mm_Vertical, symbol Connector:Conn_01x01_Pin
- added J11: EC-11, DreaM117er-keebLibrary:PinHeader_1x03_P2.54mm_Vertical, symbol Connector:Conn_01x03_Pin
- added J12: col, DreaM117er-keebLibrary:PinHeader_1x03_P2.54mm_Vertical, symbol Connector:Conn_01x03_Pin
- added JP1: JUMPER, Jumper:SolderJumper-2_P1.3mm_Open_TrianglePad1.0x1.5mm, symbol DCJACK:JUMPER
- added RE1: 1, DreaM117er-keebLibrary:RotaryEncoder_EC11, symbol DreaM117er_Library:RotaryEncoder_EC11
- added T1: AudioJack4, DreaM117er-keebLibrary:TRRS-PJ-320A, dual side x2, symbol DreaM117er_Library:TRRS
Connections:
- net GND: now also J1.3 (Pin_3), J11.2 (Pin_2), RE1.C (GND), T1.3 (R/GND)
- new net: D1.2, JP1.1, RE1.S2 (SW)
- new net 5V1: J1.1 (Pin_1), T1.1 (T/VCC)
- new net LA11: J11.1 (Pin_1), RE1.A (CLK)
- new net LB11: J11.3 (Pin_3), RE1.B (DT)
- new net LTRRS: J1.2 (Pin_2), T1.2 (R/SNL)
- new net col_re: J12.1 (Pin_1), J12.3 (Pin_3), RE1.S1 (GND)
- new net row_re: D1.1, J10.1 (Pin_1), J12.2 (Pin_2), JP1.2
- no-connect marks 0 -> 1
Other:
- moved on the sheet: H10, H11, H12, H13, H14, H15, H16, H17, H18, H19, H20, H21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
